File: source/hardware/pcb/kumand_v05.sch (EAGLE design)
At the start: 45 parts, among them IC1 ATMEGA328P_TQFP, IC2 ESP-WROOM-02, J1 3X2-SMD-DOT, X1 NX8045-CRYSTAL

Commit message: Some cosmetic touch to schematic
Parts:
- R6, R7, R8: value ? -> TBD
Connections:
- net MISO renamed S2-MISO
- net MOSI renamed S5-MOSI
- net N$11 renamed S11
- net N$12 renamed S6
- net N$13 renamed S12
- net N$16 renamed S13
- net N$17 renamed S14
- net N$18 renamed S15
- net N$23 renamed S7
- net N$5 renamed S10
- net N$6 renamed S9
- net N$7 renamed S8
- net N$8 renamed S3
- net N$9 renamed S1
- net SCK renamed S4-SCK
